File: replacement_kinesis_controller.sch (KiCad schematic (older format))
At the start: 39 parts, among them CN1 USB_general, P1 CONN_3X2, SW1 SW_PUSH, U1 MCP23018-E, U2 WS2811_RGB_LED, U3 WS2811_RGB_LED, U4 WS2811_RGB_LED, U5 WS2811_RGB_LED, U6 ATmega32U4, X1 16MHz

Commit message: More traces laid
Connections:
- net GND: no longer D4.2 (K)
- net PE6: now also D4.2 (K); no longer R7.1
- net VCC: now also R7.1
Changed lines of the file:
@@
 	1    0    0    -1
 $EndComp
-$Comp
-L GND #PWR021
-U 1 1 54C9D9EF
-P 5650 4550
-F 0 "#PWR021" H 5650 4550 30  0001 C CNN
-F 1 "GND" H 5650 4480 30  0001 C CNN
-F 2 "" H 5650 4550 60  0000 C CNN
-F 3 "" H 5650 4550 60  0000 C CNN
-	1    5650 4550
-	1    0    0    -1
-$EndComp
-Text GLabel 5650 3650 1    60   Input ~ 0
+Text GLabel 5650 4550 3    60   Input ~ 0
 PE6
 Text Label 4400 4250 0    60   ~ 0
@@
 GPB7
 $Comp
-L GND #PWR022
+L GND #PWR021
 U 1 1 54CB370B
 P 700 1150
-F 0 "#PWR022" H 700 1150 30  0001 C CNN
+F 0 "#PWR021" H 700 1150 30  0001 C CNN
 F 1 "GND" H 700 1080 30  0001 C CNN
 F 2 "" H 700 1150 60  0000 C CNN
@@
 $EndComp
 $Comp
-L VCC #PWR023
+L VCC #PWR022
 U 1 1 54CB597A
 P 750 2550
-F 0 "#PWR023" H 750 2650 30  0001 C CNN
+F 0 "#PWR022" H 750 2650 30  0001 C CNN
 F 1 "VCC" H 750 2650 30  0000 C CNN
 F 2 "" H 750 2550 60  0000 C CNN
@@
 $EndComp
 $Comp
-L GND #PWR024
+L GND #PWR023
 U 1 1 54CB76C3
 P 2900 3050
-F 0 "#PWR024" H 2900 3050 30  0001 C CNN
+F 0 "#PWR023" H 2900 3050 30  0001 C CNN
 F 1 "GND" H 2900 2980 30  0001 C CNN
 F 2 "" H 2900 3050 60  0000 C CNN
@@
 $EndComp
 $Comp
-L VCC #PWR025
+L VCC #PWR024
 U 1 1 54CB7764
 P 2900 2750
-F 0 "#PWR025" H 2900 2850 30  0001 C CNN
+F 0 "#PWR024" H 2900 2850 30  0001 C CNN
 F 1 "VCC" H 2900 2850 30  0000 C CNN
 F 2 "" H 2900 2750 60  0000 C CNN
@@
 $EndComp
 $Comp
-L VCC #PWR026
+L VCC #PWR025
 U 1 1 54D46834
 P 1600 5650
-F 0 "#PWR026" H 1600 5750 30  0001 C CNN
+F 0 "#PWR025" H 1600 5750 30  0001 C CNN
 F 1 "VCC" H 1600 5750 30  0000 C CNN
 F 2 "" H 1600 5650 60  0000 C CNN
@@
 $EndComp
 $Comp
-L GND #PWR027
+L GND #PWR026
 U 1 1 54D4A2BE
 P 1600 6250
-F 0 "#PWR027" H 1600 6250 30  0001 C CNN
+F 0 "#PWR026" H 1600 6250 30  0001 C CNN
 F 1 "GND" H 1600 6180 30  0001 C CNN
 F 2 "" H 1600 6250 60  0000 C CNN
@@
 $EndComp
 $Comp
-L VCC #PWR028
+L VCC #PWR027
 U 1 1 54DD6701
 P 3300 3450
-F 0 "#PWR028" H 3300 3550 30  0001 C CNN
+F 0 "#PWR027" H 3300 3550 30  0001 C CNN
 F 1 "VCC" H 3300 3550 30  0000 C CNN
 F 2 "" H 3300 3450 60  0000 C CNN
@@
 Connection ~ 1500 5450
 $Comp
-L VCC #PWR029
+L VCC #PWR028
 U 1 1 54E6DA2C
 P 8900 5600
-F 0 "#PWR029" H 8900 5700 30  0001 C CNN
+F 0 "#PWR028" H 8900 5700 30  0001 C CNN
 F 1 "VCC" H 8900 5700 30  0000 C CNN
 F 2 "" H 8900 5600 60  0000 C CNN
@@
 $EndComp
 $Comp
-L GND #PWR030
+L GND #PWR029
 U 1 1 54E6DBB8
 P 8900 6050
-F 0 "#PWR030" H 8900 6050 30  0001 C CNN
+F 0 "#PWR029" H 8900 6050 30  0001 C CNN
 F 1 "GND" H 8900 5980 30  0001 C CNN
 F 2 "" H 8900 6050 60  0000 C CNN
@@
 $EndSheet
 $Comp
-L VCC #PWR031
+L VCC #PWR030
 U 1 1 54E71458
 P 1250 3750
-F 0 "#PWR031" H 1250 3850 30  0001 C CNN
+F 0 "#PWR030" H 1250 3850 30  0001 C CNN
 F 1 "VCC" H 1250 3850 30  0000 C CNN
 F 2 "" H 1250 3750 60  0000 C CNN
@@
 $EndComp
 $Comp
-L GND #PWR032
+L GND #PWR031
 U 1 1 54E7145E
 P 1250 4200
-F 0 "#PWR032" H 1250 4200 30  0001 C CNN
+F 0 "#PWR031" H 1250 4200 30  0001 C CNN
 F 1 "GND" H 1250 4130 30  0001 C CNN
 F 2 "" H 1250 4200 60  0000 C CNN
@@
 $EndComp
 $Comp
-L GND #PWR033
+L GND #PWR032
 U 1 1 54E8CE58
 P 7600 1650
-F 0 "#PWR033" H 7600 1650 30  0001 C CNN
+F 0 "#PWR032" H 7600 1650 30  0001 C CNN
 F 1 "GND" H 7600 1580 30  0001 C CNN
 F 2 "" H 7600 1650 60  0000 C CNN
@@
 Wire Wire Line
 	8050 2550 8050 2400
+$Comp
+L VCC #PWR033
+U 1 1 54FB6693
+P 5650 3650
+F 0 "#PWR033" H 5650 3750 30  0001 C CNN
+F 1 "VCC" H 5650 3750 30  0000 C CNN
+F 2 "" H 5650 3650 60  0000 C CNN
+F 3 "" H 5650 3650 60  0000 C CNN
+	1    5650 3650
+	1    0    0    -1
+$EndComp
 $EndSCHEMATC
