File: breakouts.sch (KiCad schematic (older format))
At the start: 26 parts

Commit message: Add annotations to parts
Parts:
- gave numbers to parts that had none: 26
Changed lines of the file:
@@
 COL_11
 $Comp
-L CONN_6 P?
+L CONN_6 P13
 U 1 1 54E55166
 P 4500 3200
-F 0 "P?" V 4450 3200 60  0000 C CNN
+F 0 "P13" V 4450 3200 60  0000 C CNN
 F 1 "CONN_6" V 4550 3200 60  0000 C CNN
 F 2 "" H 4500 3200 60  0000 C CNN
@@
 $EndComp
 $Comp
-L CONN_6 P?
+L CONN_6 P9
 U 1 1 54E5516D
 P 2250 3200
-F 0 "P?" V 2200 3200 60  0000 C CNN
+F 0 "P9" V 2200 3200 60  0000 C CNN
 F 1 "CONN_6" V 2300 3200 60  0000 C CNN
 F 2 "" H 2250 3200 60  0000 C CNN
@@
 $EndComp
 $Comp
-L CONN_8 P?
+L CONN_8 P14
 U 1 1 54E55174
 P 4500 4000
-F 0 "P?" V 4450 4000 60  0000 C CNN
+F 0 "P14" V 4450 4000 60  0000 C CNN
 F 1 "CONN_8" V 4550 4000 60  0000 C CNN
 F 2 "" H 4500 4000 60  0000 C CNN
@@
 $EndComp
 $Comp
-L CONN_8 P?
+L CONN_8 P10
 U 1 1 54E5517B
 P 2250 4000
-F 0 "P?" V 2200 4000 60  0000 C CNN
+F 0 "P10" V 2200 4000 60  0000 C CNN
 F 1 "CONN_8" V 2300 4000 60  0000 C CNN
 F 2 "" H 2250 4000 60  0000 C CNN
@@
 PD1
 $Comp
-L GND #PWR?
+L GND #PWR35
 U 1 1 54E556E0
 P 2450 6050
-F 0 "#PWR?" H 2450 6050 30  0001 C CNN
+F 0 "#PWR35" H 2450 6050 30  0001 C CNN
 F 1 "GND" H 2450 5980 30  0001 C CNN
 F 2 "" H 2450 6050 60  0000 C CNN
@@
 $EndComp
 $Comp
-L GND #PWR?
+L GND #PWR37
 U 1 1 54E556E6
 P 4750 6050
-F 0 "#PWR?" H 4750 6050 30  0001 C CNN
+F 0 "#PWR37" H 4750 6050 30  0001 C CNN
 F 1 "GND" H 4750 5980 30  0001 C CNN
 F 2 "" H 4750 6050 60  0000 C CNN
@@
 $EndComp
 $Comp
-L VCC #PWR?
+L VCC #PWR34
 U 1 1 54E556EC
 P 2450 5800
-F 0 "#PWR?" H 2450 5900 30  0001 C CNN
+F 0 "#PWR34" H 2450 5900 30  0001 C CNN
 F 1 "VCC" H 2450 5900 30  0000 C CNN
 F 2 "" H 2450 5800 60  0000 C CNN
@@
 $EndComp
 $Comp
-L VCC #PWR?
+L VCC #PWR36
 U 1 1 54E556F2
 P 4750 5800
-F 0 "#PWR?" H 4750 5900 30  0001 C CNN
+F 0 "#PWR36" H 4750 5900 30  0001 C CNN
 F 1 "VCC" H 4750 5900 30  0000 C CNN
 F 2 "" H 4750 5800 60  0000 C CNN
@@
 	4750 5900 4750 5800
 $Comp
-L +5V #PWR?
+L +5V #PWR39
 U 1 1 54E569F6
 P 6250 2900
-F 0 "#PWR?" H 6250 2990 20  0001 C CNN
+F 0 "#PWR39" H 6250 2990 20  0001 C CNN
 F 1 "+5V" H 6250 2990 30  0000 C CNN
 F 2 "" H 6250 2900 60  0000 C CNN
@@
 PB4
 $Comp
-L GND #PWR?
+L GND #PWR38
 U 1 1 54E56A09
 P 5700 4500
-F 0 "#PWR?" H 5700 4500 30  0001 C CNN
+F 0 "#PWR38" H 5700 4500 30  0001 C CNN
 F 1 "GND" H 5700 4430 30  0001 C CNN
 F 2 "" H 5700 4500 60  0000 C CNN
@@
 PE6
 $Comp
-L +3.3V #PWR?
+L +3.3V #PWR40
 U 1 1 54E56A23
 P 7450 2900
-F 0 "#PWR?" H 7450 2860 30  0001 C CNN
+F 0 "#PWR40" H 7450 2860 30  0001 C CNN
 F 1 "+3.3V" H 7450 3010 30  0000 C CNN
 F 2 "" H 7450 2900 60  0000 C CNN
@@
 	6250 3000 6250 2900
 $Comp
-L CONN_16 P?
+L CONN_16 P17
 U 1 1 54E56DFC
 P 7100 3750
-F 0 "P?" V 7060 3750 60  0000 C CNN
+F 0 "P17" V 7060 3750 60  0000 C CNN
 F 1 "CONN_16" V 7180 3750 60  0000 C CNN
 F 2 "" H 7100 3750 60  0000 C CNN
@@
 $EndComp
 $Comp
-L CONN_16 P?
+L CONN_16 P16
 U 1 1 54E56E45
 P 6600 3750
-F 0 "P?" V 6560 3750 60  0000 C CNN
+F 0 "P16" V 6560 3750 60  0000 C CNN
 F 1 "CONN_16" V 6680 3750 60  0000 C CNN
 F 2 "" H 6600 3750 60  0000 C CNN
@@
 	7450 4400 8000 4400
 $Comp
-L GND #PWR?
+L GND #PWR42
 U 1 1 54E56FF9
 P 8000 4500
-F 0 "#PWR?" H 8000 4500 30  0001 C CNN
+F 0 "#PWR42" H 8000 4500 30  0001 C CNN
 F 1 "GND" H 8000 4430 30  0001 C CNN
 F 2 "" H 8000 4500 60  0000 C CNN
@@
 	8000 4400 8000 4500
 $Comp
-L VCC #PWR?
+L VCC #PWR41
 U 1 1 54E42A55
 P 7800 4500
-F 0 "#PWR?" H 7800 4600 30  0001 C CNN
+F 0 "#PWR41" H 7800 4600 30  0001 C CNN
 F 1 "VCC" H 7800 4600 30  0000 C CNN
 F 2 "" H 7800 4500 60  0000 C CNN
@@
 $EndComp
 $Comp
-L CONN_6 P?
+L CONN_6 P23
 U 1 1 54E5EB00
 P 10600 4900
-F 0 "P?" V 10550 4900 60  0000 C CNN
+F 0 "P23" V 10550 4900 60  0000 C CNN
 F 1 "SMIRF" V 10650 4900 60  0000 C CNN
 F 2 "" H 10600 4900 60  0000 C CNN
@@
 W_NCTS
 $Comp
-L VCC #PWR?
+L VCC #PWR47
 U 1 1 54E5EB0B
 P 10050 5050
-F 0 "#PWR?" H 10050 5150 30  0001 C CNN
+F 0 "#PWR47" H 10050 5150 30  0001 C CNN
 F 1 "VCC" H 10050 5150 30  0000 C CNN
 F 2 "" H 10050 5050 60  0000 C CNN
@@
 $EndComp
 $Comp
-L GND #PWR?
+L GND #PWR46
 U 1 1 54E5EB11
 P 10050 4950
-F 0 "#PWR?" H 10050 4950 30  0001 C CNN
+F 0 "#PWR46" H 10050 4950 30  0001 C CNN
 F 1 "GND" H 10050 4880 30  0001 C CNN
 F 2 "" H 10050 4950 60  0000 C CNN
@@
 $EndComp
 $Comp
-L CONN_6 P?
+L CONN_6 P22
 U 1 1 54E5EB17
 P 10600 4100
-F 0 "P?" V 10550 4100 60  0000 C CNN
+F 0 "P22" V 10550 4100 60  0000 C CNN
 F 1 "IO" V 10650 4100 60  0000 C CNN
 F 2 "" H 10600 4100 60  0000 C CNN
@@
 W_PIO3
 $Comp
-L CONN_4 P?
+L CONN_4 P21
 U 1 1 54E5EB24
 P 10600 3400
-F 0 "P?" V 10550 3400 50  0000 C CNN
+F 0 "P21" V 10550 3400 50  0000 C CNN
 F 1 "SPI" V 10650 3400 50  0000 C CNN
 F 2 "" H 10600 3400 60  0000 C CNN
@@
 $EndComp
 $Comp
-L CONN_4 P?
+L CONN_4 P20
 U 1 1 54E5EB2B
 P 10600 2800
-F 0 "P?" V 10550 2800 50  0000 C CNN
+F 0 "P20" V 10550 2800 50  0000 C CNN
 F 1 "UART" V 10650 2800 50  0000 C CNN
 F 2 "" H 10600 2800 60  0000 C CNN
@@
 $EndComp
 $Comp
-L CONN_4 P?
+L CONN_4 P19
 U 1 1 54E5EB32
 P 10600 2200
-F 0 "P?" V 10550 2200 50  0000 C CNN
+F 0 "P19" V 10550 2200 50  0000 C CNN
 F 1 "PCM" V 10650 2200 50  0000 C CNN
 F 2 "" H 10600 2200 60  0000 C CNN
@@
 $EndComp
 $Comp
-L CONN_4 P?
+L CONN_4 P18
 U 1 1 54E5EB39
 P 10600 1600
-F 0 "P?" V 10550 1600 50  0000 C CNN
+F 0 "P18" V 10550 1600 50  0000 C CNN
 F 1 "POWER" V 10650 1600 50  0000 C CNN
 F 2 "" H 10600 1600 60  0000 C CNN
@@
 W_RESET
 $Comp
-L VCC #PWR?
+L VCC #PWR45
 U 1 1 54E5EB4D
 P 10050 1650
-F 0 "#PWR?" H 10050 1750 30  0001 C CNN
+F 0 "#PWR45" H 10050 1750 30  0001 C CNN
 F 1 "VCC" H 10050 1750 30  0000 C CNN
 F 2 "" H 10050 1650 60  0000 C CNN
@@
 $EndComp
 $Comp
-L +5V #PWR?
+L +5V #PWR44
 U 1 1 54E5EB53
 P 10050 1550
-F 0 "#PWR?" H 10050 1640 20  0001 C CNN
+F 0 "#PWR44" H 10050 1640 20  0001 C CNN
 F 1 "+5V" H 10050 1640 30  0000 C CNN
 F 2 "" H 10050 1550 60  0000 C CNN
@@
 $EndComp
 $Comp
-L GND #PWR?
+L GND #PWR43
 U 1 1 54E5EB59
 P 10050 1450
-F 0 "#PWR?" H 10050 1450 30  0001 C CNN
+F 0 "#PWR43" H 10050 1450 30  0001 C CNN
 F 1 "GND" H 10050 1380 30  0001 C CNN
 F 2 "" H 10050 1450 60  0000 C CNN
@@
 	10250 1750 10050 1750
 $Comp
-L CONN_5X2 P?
+L CONN_5X2 P8
 U 1 1 54E5FC1B
 P 1700 1800
-F 0 "P?" H 1700 2100 60  0000 C CNN
+F 0 "P8" H 1700 2100 60  0000 C CNN
 F 1 "CONN_5X2" V 1700 1800 50  0000 C CNN
 F 2 "" H 1700 1800 60  0000 C CNN
@@
 $EndComp
 $Comp
-L DIODE D?
+L DIODE D5
 U 1 1 54E5FC22
 P 2500 1200
-F 0 "D?" H 2500 1300 40  0000 C CNN
+F 0 "D5" H 2500 1300 40  0000 C CNN
 F 1 "DIODE" H 2500 1100 40  0000 C CNN
 F 2 "" H 2500 1200 60  0000 C CNN
@@
 $EndComp
 $Comp
-L DIODE D?
+L DIODE D9
 U 1 1 54E5FC29
 P 2500 2400
-F 0 "D?" H 2500 2500 40  0000 C CNN
+F 0 "D9" H 2500 2500 40  0000 C CNN
 F 1 "DIODE" H 2500 2300 40  0000 C CNN
 F 2 "" H 2500 2400 60  0000 C CNN
@@
 $EndComp
 $Comp
-L DIODE D?
+L DIODE D8
 U 1 1 54E5FC30
 P 2500 2100
-F 0 "D?" H 2500 2200 40  0000 C CNN
+F 0 "D8" H 2500 2200 40  0000 C CNN
 F 1 "DIODE" H 2500 2000 40  0000 C CNN
 F 2 "" H 2500 2100 60  0000 C CNN
@@
 $EndComp
 $Comp
-L DIODE D?
+L DIODE D6
 U 1 1 54E5FC37
 P 2500 1500
-F 0 "D?" H 2500 1600 40  0000 C CNN
+F 0 "D6" H 2500 1600 40  0000 C CNN
 F 1 "DIODE" H 2500 1400 40  0000 C CNN
 F 2 "" H 2500 1500 60  0000 C CNN
@@
 $EndComp
 $Comp
-L DIODE D?
+L DIODE D7
 U 1 1 54E5FC3E
 P 2500 1800
-F 0 "D?" H 2500 1900 40  0000 C CNN
+F 0 "D7" H 2500 1900 40  0000 C CNN
 F 1 "DIODE" H 2500 1700 40  0000 C CNN
 F 2 "" H 2500 1800 60  0000 C CNN
@@
 	1200 1600 1300 1600
 $Comp
-L CONN_5X2 P?
+L CONN_5X2 P15
 U 1 1 54E5FC70
 P 4900 1800
-F 0 "P?" H 4900 2100 60  0000 C CNN
+F 0 "P15" H 4900 2100 60  0000 C CNN
 F 1 "CONN_5X2" V 4900 1800 50  0000 C CNN
 F 2 "" H 4900 1800 60  0000 C CNN
@@
 $EndComp
 $Comp
-L DIODE D?
+L DIODE D10
 U 1 1 54E5FC77
 P 4100 1200
-F 0 "D?" H 4100 1300 40  0000 C CNN
+F 0 "D10" H 4100 1300 40  0000 C CNN
 F 1 "DIODE" H 4100 1100 40  0000 C CNN
 F 2 "" H 4100 1200 60  0000 C CNN
@@
 $EndComp
 $Comp
-L DIODE D?
+L DIODE D14
 U 1 1 54E5FC7E
 P 4100 2400
-F 0 "D?" H 4100 2500 40  0000 C CNN
+F 0 "D14" H 4100 2500 40  0000 C CNN
 F 1 "DIODE" H 4100 2300 40  0000 C CNN
 F 2 "" H 4100 2400 60  0000 C CNN
@@
 $EndComp
 $Comp
-L DIODE D?
+L DIODE D13
 U 1 1 54E5FC85
 P 4100 2100
-F 0 "D?" H 4100 2200 40  0000 C CNN
+F 0 "D13" H 4100 2200 40  0000 C CNN
 F 1 "DIODE" H 4100 2000 40  0000 C CNN
 F 2 "" H 4100 2100 60  0000 C CNN
@@
 $EndComp
 $Comp
-L DIODE D?
+L DIODE D11
 U 1 1 54E5FC8C
 P 4100 1500
-F 0 "D?" H 4100 1600 40  0000 C CNN
+F 0 "D11" H 4100 1600 40  0000 C CNN
 F 1 "DIODE" H 4100 1400 40  0000 C CNN
 F 2 "" H 4100 1500 60  0000 C CNN
@@
 $EndComp
 $Comp
-L DIODE D?
+L DIODE D12
 U 1 1 54E5FC93
 P 4100 1800
-F 0 "D?" H 4100 1900 40  0000 C CNN
+F 0 "D12" H 4100 1900 40  0000 C CNN
 F 1 "DIODE" H 4100 1700 40  0000 C CNN
 F 2 "" H 4100 1800 60  0000 C CNN
@@
 COL_11
 $Comp
-L CONN_5 P?
+L CONN_5 P11
 U 1 1 54E803DF
 P 3350 6100
-F 0 "P?" V 3300 6100 50  0000 C CNN
+F 0 "P11" V 3300 6100 50  0000 C CNN
 F 1 "CONN_5" V 3400 6100 50  0000 C CNN
 F 2 "" H 3350 6100 60  0000 C CNN
@@
 $EndComp
 $Comp
-L CONN_5 P?
+L CONN_5 P12
 U 1 1 54E80505
 P 3850 6100
-F 0 "P?" V 3800 6100 50  0000 C CNN
+F 0 "P12" V 3800 6100 50  0000 C CNN
 F 1 "CONN_5" V 3900 6100 50  0000 C CNN
 F 2 "" H 3850 6100 60  0000 C CNN

Commit message: WT12 breakout headers are now in place
Parts:
- added P?: USB, symbol CONN_2
- P15, P8: footprint (none) -> replacement_kinesis_controller:Pin_Header_Staggered_Straight_2x05
- P16, P17: footprint (none) -> replacement_kinesis_controller:Pin_Header_Staggered_Straight_1x16
- P18, P19, P20, P21: footprint (none) -> replacement_kinesis_controller:Pin_Header_Staggered_Straight_1x04
- P22, P23, P9: footprint (none) -> replacement_kinesis_controller:Pin_Header_Staggered_Straight_1x06
Connections:
- new net W_USB_D+: P?.2 (PM)
- new net W_USB_D-: P?.1 (P1)
Changed lines of the file:
@@
 F 0 "P13" V 4450 3200 60  0000 C CNN
 F 1 "CONN_6" V 4550 3200 60  0000 C CNN
-F 2 "" H 4500 3200 60  0000 C CNN
+F 2 "" H 4500 3200 60  0001 C CNN
 F 3 "" H 4500 3200 60  0000 C CNN
 	1    4500 3200
@@
 F 0 "P9" V 2200 3200 60  0000 C CNN
 F 1 "CONN_6" V 2300 3200 60  0000 C CNN
-F 2 "" H 2250 3200 60  0000 C CNN
+F 2 "replacement_kinesis_controller:Pin_Header_Staggered_Straight_1x06" H 2250 3200 60  0001 C CNN
 F 3 "" H 2250 3200 60  0000 C CNN
 	1    2250 3200
@@
 F 0 "P14" V 4450 4000 60  0000 C CNN
 F 1 "CONN_8" V 4550 4000 60  0000 C CNN
-F 2 "" H 4500 4000 60  0000 C CNN
+F 2 "" H 4500 4000 60  0001 C CNN
 F 3 "" H 4500 4000 60  0000 C CNN
 	1    4500 4000
@@
 F 0 "P10" V 2200 4000 60  0000 C CNN
 F 1 "CONN_8" V 2300 4000 60  0000 C CNN
-F 2 "" H 2250 4000 60  0000 C CNN
+F 2 "" H 2250 4000 60  0001 C CNN
 F 3 "" H 2250 4000 60  0000 C CNN
 	1    2250 4000
@@
 F 0 "P17" V 7060 3750 60  0000 C CNN
 F 1 "CONN_16" V 7180 3750 60  0000 C CNN
-F 2 "" H 7100 3750 60  0000 C CNN
+F 2 "replacement_kinesis_controller:Pin_Header_Staggered_Straight_1x16" H 7100 3750 60  0001 C CNN
 F 3 "" H 7100 3750 60  0000 C CNN
 	1    7100 3750
@@
 F 0 "P16" V 6560 3750 60  0000 C CNN
 F 1 "CONN_16" V 6680 3750 60  0000 C CNN
-F 2 "" H 6600 3750 60  0000 C CNN
+F 2 "replacement_kinesis_controller:Pin_Header_Staggered_Straight_1x16" H 6600 3750 60  0001 C CNN
 F 3 "" H 6600 3750 60  0000 C CNN
 	1    6600 3750
@@
 F 0 "P23" V 10550 4900 60  0000 C CNN
 F 1 "SMIRF" V 10650 4900 60  0000 C CNN
-F 2 "" H 10600 4900 60  0000 C CNN
+F 2 "replacement_kinesis_controller:Pin_Header_Staggered_Straight_1x06" H 10600 4900 60  0001 C CNN
 F 3 "" H 10600 4900 60  0000 C CNN
 	1    10600 4900
@@
 F 0 "P22" V 10550 4100 60  0000 C CNN
 F 1 "IO" V 10650 4100 60  0000 C CNN
-F 2 "" H 10600 4100 60  0000 C CNN
+F 2 "replacement_kinesis_controller:Pin_Header_Staggered_Straight_1x06" H 10600 4100 60  0001 C CNN
 F 3 "" H 10600 4100 60  0000 C CNN
 	1    10600 4100
@@
 F 0 "P21" V 10550 3400 50  0000 C CNN
 F 1 "SPI" V 10650 3400 50  0000 C CNN
-F 2 "" H 10600 3400 60  0000 C CNN
+F 2 "replacement_kinesis_controller:Pin_Header_Staggered_Straight_1x04" H 10600 3400 60  0001 C CNN
 F 3 "" H 10600 3400 60  0000 C CNN
 	1    10600 3400
@@
 F 0 "P20" V 10550 2800 50  0000 C CNN
 F 1 "UART" V 10650 2800 50  0000 C CNN
-F 2 "" H 10600 2800 60  0000 C CNN
+F 2 "replacement_kinesis_controller:Pin_Header_Staggered_Straight_1x04" H 10600 2800 60  0001 C CNN
 F 3 "" H 10600 2800 60  0000 C CNN
 	1    10600 2800
@@
 F 0 "P19" V 10550 2200 50  0000 C CNN
 F 1 "PCM" V 10650 2200 50  0000 C CNN
-F 2 "" H 10600 2200 60  0000 C CNN
+F 2 "replacement_kinesis_controller:Pin_Header_Staggered_Straight_1x04" H 10600 2200 60  0001 C CNN
 F 3 "" H 10600 2200 60  0000 C CNN
 	1    10600 2200
@@
 F 0 "P18" V 10550 1600 50  0000 C CNN
 F 1 "POWER" V 10650 1600 50  0000 C CNN
-F 2 "" H 10600 1600 60  0000 C CNN
+F 2 "replacement_kinesis_controller:Pin_Header_Staggered_Straight_1x04" H 10600 1600 60  0001 C CNN
 F 3 "" H 10600 1600 60  0000 C CNN
 	1    10600 1600
@@
 F 0 "P8" H 1700 2100 60  0000 C CNN
 F 1 "CONN_5X2" V 1700 1800 50  0000 C CNN
-F 2 "" H 1700 1800 60  0000 C CNN
+F 2 "replacement_kinesis_controller:Pin_Header_Staggered_Straight_2x05" H 1700 1800 60  0001 C CNN
 F 3 "" H 1700 1800 60  0000 C CNN
 	1    1700 1800
@@
 F 0 "D5" H 2500 1300 40  0000 C CNN
 F 1 "DIODE" H 2500 1100 40  0000 C CNN
-F 2 "" H 2500 1200 60  0000 C CNN
+F 2 "" H 2500 1200 60  0001 C CNN
 F 3 "" H 2500 1200 60  0000 C CNN
 	1    2500 1200
@@
 F 0 "D9" H 2500 2500 40  0000 C CNN
 F 1 "DIODE" H 2500 2300 40  0000 C CNN
-F 2 "" H 2500 2400 60  0000 C CNN
+F 2 "" H 2500 2400 60  0001 C CNN
 F 3 "" H 2500 2400 60  0000 C CNN
 	1    2500 2400
@@
 F 0 "D8" H 2500 2200 40  0000 C CNN
 F 1 "DIODE" H 2500 2000 40  0000 C CNN
-F 2 "" H 2500 2100 60  0000 C CNN
+F 2 "" H 2500 2100 60  0001 C CNN
 F 3 "" H 2500 2100 60  0000 C CNN
 	1    2500 2100
@@
 F 0 "D6" H 2500 1600 40  0000 C CNN
 F 1 "DIODE" H 2500 1400 40  0000 C CNN
-F 2 "" H 2500 1500 60  0000 C CNN
+F 2 "" H 2500 1500 60  0001 C CNN
 F 3 "" H 2500 1500 60  0000 C CNN
 	1    2500 1500
@@
 F 0 "D7" H 2500 1900 40  0000 C CNN
 F 1 "DIODE" H 2500 1700 40  0000 C CNN
-F 2 "" H 2500 1800 60  0000 C CNN
+F 2 "" H 2500 1800 60  0001 C CNN
 F 3 "" H 2500 1800 60  0000 C CNN
 	1    2500 1800
@@
 F 0 "P15" H 4900 2100 60  0000 C CNN
 F 1 "CONN_5X2" V 4900 1800 50  0000 C CNN
-F 2 "" H 4900 1800 60  0000 C CNN
+F 2 "replacement_kinesis_controller:Pin_Header_Staggered_Straight_2x05" H 4900 1800 60  0001 C CNN
 F 3 "" H 4900 1800 60  0000 C CNN
 	1    4900 1800
@@
 F 0 "D10" H 4100 1300 40  0000 C CNN
 F 1 "DIODE" H 4100 1100 40  0000 C CNN
-F 2 "" H 4100 1200 60  0000 C CNN
+F 2 "" H 4100 1200 60  0001 C CNN
 F 3 "" H 4100 1200 60  0000 C CNN
 	1    4100 1200
@@
 F 0 "D14" H 4100 2500 40  0000 C CNN
 F 1 "DIODE" H 4100 2300 40  0000 C CNN
-F 2 "" H 4100 2400 60  0000 C CNN
+F 2 "" H 4100 2400 60  0001 C CNN
 F 3 "" H 4100 2400 60  0000 C CNN
 	1    4100 2400
@@
 F 0 "D13" H 4100 2200 40  0000 C CNN
 F 1 "DIODE" H 4100 2000 40  0000 C CNN
-F 2 "" H 4100 2100 60  0000 C CNN
+F 2 "" H 4100 2100 60  0001 C CNN
 F 3 "" H 4100 2100 60  0000 C CNN
 	1    4100 2100
@@
 F 0 "D11" H 4100 1600 40  0000 C CNN
 F 1 "DIODE" H 4100 1400 40  0000 C CNN
-F 2 "" H 4100 1500 60  0000 C CNN
+F 2 "" H 4100 1500 60  0001 C CNN
 F 3 "" H 4100 1500 60  0000 C CNN
 	1    4100 1500
@@
 F 0 "D12" H 4100 1900 40  0000 C CNN
 F 1 "DIODE" H 4100 1700 40  0000 C CNN
-F 2 "" H 4100 1800 60  0000 C CNN
+F 2 "" H 4100 1800 60  0001 C CNN
 F 3 "" H 4100 1800 60  0000 C CNN
 	1    4100 1800
@@
 F 0 "P11" V 3300 6100 50  0000 C CNN
 F 1 "CONN_5" V 3400 6100 50  0000 C CNN
-F 2 "" H 3350 6100 60  0000 C CNN
+F 2 "" H 3350 6100 60  0001 C CNN
 F 3 "" H 3350 6100 60  0000 C CNN
 	1    3350 6100
@@
 F 0 "P12" V 3800 6100 50  0000 C CNN
 F 1 "CONN_5" V 3900 6100 50  0000 C CNN
-F 2 "" H 3850 6100 60  0000 C CNN
+F 2 "" H 3850 6100 60  0001 C CNN
 F 3 "" H 3850 6100 60  0000 C CNN
 	1    3850 6100
@@
 Text Notes 9450 1250 0    60   ~ 0
 5V and VCC here are from the\nWT12 breakout board's built in\nregulator. Will this cause problems?
+$Comp
+L CONN_2 P?
+U 1 1 54EA265F
+P 10600 5600
+F 0 "P?" V 10550 5600 40  0000 C CNN
+F 1 "USB" V 10650 5600 40  0000 C CNN
+F 2 "" H 10600 5600 60  0000 C CNN
+F 3 "" H 10600 5600 60  0000 C CNN
+	1    10600 5600
+	1    0    0    -1
+$EndComp
+Text GLabel 10050 5700 0    60   Input ~ 0
+W_USB_D+
+Text GLabel 10050 5500 0    60   Input ~ 0
+W_USB_D-
+Wire Wire Line
+	10050 5500 10250 5500
+Wire Wire Line
+	10050 5700 10250 5700
 $EndSCHEMATC

Commit message: Add footprints to regular diodes
Parts:
- D10, D11, D12, D13, D14, D5, D6, D7, D8, D9: footprint (none) -> replacement_kinesis_controller:SOD-323_Handsolder
Changed lines of the file:
@@
 F 0 "D5" H 2500 1300 40  0000 C CNN
 F 1 "DIODE" H 2500 1100 40  0000 C CNN
-F 2 "" H 2500 1200 60  0001 C CNN
+F 2 "replacement_kinesis_controller:SOD-323_Handsolder" H 2500 1200 60  0001 C CNN
 F 3 "" H 2500 1200 60  0000 C CNN
 	1    2500 1200
@@
 F 0 "D9" H 2500 2500 40  0000 C CNN
 F 1 "DIODE" H 2500 2300 40  0000 C CNN
-F 2 "" H 2500 2400 60  0001 C CNN
+F 2 "replacement_kinesis_controller:SOD-323_Handsolder" H 2500 2400 60  0001 C CNN
 F 3 "" H 2500 2400 60  0000 C CNN
 	1    2500 2400
@@
 F 0 "D8" H 2500 2200 40  0000 C CNN
 F 1 "DIODE" H 2500 2000 40  0000 C CNN
-F 2 "" H 2500 2100 60  0001 C CNN
+F 2 "replacement_kinesis_controller:SOD-323_Handsolder" H 2500 2100 60  0001 C CNN
 F 3 "" H 2500 2100 60  0000 C CNN
 	1    2500 2100
@@
 F 0 "D6" H 2500 1600 40  0000 C CNN
 F 1 "DIODE" H 2500 1400 40  0000 C CNN
-F 2 "" H 2500 1500 60  0001 C CNN
+F 2 "replacement_kinesis_controller:SOD-323_Handsolder" H 2500 1500 60  0001 C CNN
 F 3 "" H 2500 1500 60  0000 C CNN
 	1    2500 1500
@@
 F 0 "D7" H 2500 1900 40  0000 C CNN
 F 1 "DIODE" H 2500 1700 40  0000 C CNN
-F 2 "" H 2500 1800 60  0001 C CNN
+F 2 "replacement_kinesis_controller:SOD-323_Handsolder" H 2500 1800 60  0001 C CNN
 F 3 "" H 2500 1800 60  0000 C CNN
 	1    2500 1800
@@
 F 0 "D10" H 4100 1300 40  0000 C CNN
 F 1 "DIODE" H 4100 1100 40  0000 C CNN
-F 2 "" H 4100 1200 60  0001 C CNN
+F 2 "replacement_kinesis_controller:SOD-323_Handsolder" H 4100 1200 60  0001 C CNN
 F 3 "" H 4100 1200 60  0000 C CNN
 	1    4100 1200
@@
 F 0 "D14" H 4100 2500 40  0000 C CNN
 F 1 "DIODE" H 4100 2300 40  0000 C CNN
-F 2 "" H 4100 2400 60  0001 C CNN
+F 2 "replacement_kinesis_controller:SOD-323_Handsolder" H 4100 2400 60  0001 C CNN
 F 3 "" H 4100 2400 60  0000 C CNN
 	1    4100 2400
@@
 F 0 "D13" H 4100 2200 40  0000 C CNN
 F 1 "DIODE" H 4100 2000 40  0000 C CNN
-F 2 "" H 4100 2100 60  0001 C CNN
+F 2 "replacement_kinesis_controller:SOD-323_Handsolder" H 4100 2100 60  0001 C CNN
 F 3 "" H 4100 2100 60  0000 C CNN
 	1    4100 2100
@@
 F 0 "D11" H 4100 1600 40  0000 C CNN
 F 1 "DIODE" H 4100 1400 40  0000 C CNN
-F 2 "" H 4100 1500 60  0001 C CNN
+F 2 "replacement_kinesis_controller:SOD-323_Handsolder" H 4100 1500 60  0001 C CNN
 F 3 "" H 4100 1500 60  0000 C CNN
 	1    4100 1500
@@
 F 0 "D12" H 4100 1900 40  0000 C CNN
 F 1 "DIODE" H 4100 1700 40  0000 C CNN
-F 2 "" H 4100 1800 60  0001 C CNN
+F 2 "replacement_kinesis_controller:SOD-323_Handsolder" H 4100 1800 60  0001 C CNN
 F 3 "" H 4100 1800 60  0000 C CNN
 	1    4100 1800

Commit message: More footprints
Parts:
- P10, P14: footprint (none) -> replacement_kinesis_controller:Pin_Header_Staggered_Straight_1x08
- P11, P12: footprint (none) -> replacement_kinesis_controller:Pin_Header_Staggered_Straight_1x05
- P13: footprint (none) -> replacement_kinesis_controller:Pin_Header_Staggered_Straight_1x06
Changed lines of the file:
@@
 F 0 "P13" V 4450 3200 60  0000 C CNN
 F 1 "CONN_6" V 4550 3200 60  0000 C CNN
-F 2 "" H 4500 3200 60  0001 C CNN
+F 2 "replacement_kinesis_controller:Pin_Header_Staggered_Straight_1x06" H 4500 3200 60  0001 C CNN
 F 3 "" H 4500 3200 60  0000 C CNN
 	1    4500 3200
@@
 F 0 "P14" V 4450 4000 60  0000 C CNN
 F 1 "CONN_8" V 4550 4000 60  0000 C CNN
-F 2 "" H 4500 4000 60  0001 C CNN
+F 2 "replacement_kinesis_controller:Pin_Header_Staggered_Straight_1x08" H 4500 4000 60  0001 C CNN
 F 3 "" H 4500 4000 60  0000 C CNN
 	1    4500 4000
@@
 F 0 "P10" V 2200 4000 60  0000 C CNN
 F 1 "CONN_8" V 2300 4000 60  0000 C CNN
-F 2 "" H 2250 4000 60  0001 C CNN
+F 2 "replacement_kinesis_controller:Pin_Header_Staggered_Straight_1x08" H 2250 4000 60  0001 C CNN
 F 3 "" H 2250 4000 60  0000 C CNN
 	1    2250 4000
@@
 F 0 "P11" V 3300 6100 50  0000 C CNN
 F 1 "CONN_5" V 3400 6100 50  0000 C CNN
-F 2 "" H 3350 6100 60  0001 C CNN
+F 2 "replacement_kinesis_controller:Pin_Header_Staggered_Straight_1x05" H 3350 6100 60  0001 C CNN
 F 3 "" H 3350 6100 60  0000 C CNN
 	1    3350 6100
@@
 F 0 "P12" V 3800 6100 50  0000 C CNN
 F 1 "CONN_5" V 3900 6100 50  0000 C CNN
-F 2 "" H 3850 6100 60  0001 C CNN
+F 2 "replacement_kinesis_controller:Pin_Header_Staggered_Straight_1x05" H 3850 6100 60  0001 C CNN
 F 3 "" H 3850 6100 60  0000 C CNN
 	1    3850 6100
